File: kicad/sensor_cluster.kicad_sch (KiCad schematic)
At the start: 19 parts, among them J11 B2B-XH-ALFSN, J12 B4B-XH-A, J9 B2B-XH-ALFSN, U5 TPS92200D1DDCR, U6 TPS92200D1DDCR

Commit message: finish first pcb revision
Parts:
- C37, C39, C42, C43: footprint (none) -> Capacitor_SMD:C_0201_0603Metric
- C38, C40, C41, C44: footprint (none) -> Capacitor_SMD:C_0603_1608Metric
- J11, J9: footprint (none) -> B2B-XH-A:CONN_B2B-XH-ALFSN_JST
- L2, L4: footprint (none) -> ETQP3M4R7KVN:ETQP3M1R0KVN
- R16, R27, R30, R31: footprint (none) -> Resistor_SMD:R_0201_0603Metric
- U5, U6: footprint (none) -> TPS92200D1DDCR:DDC0006A_N
Changed lines of the file:
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@@
 			)
 		)
-		(property "Footprint" ""
+		(property "Footprint" "Capacitor_SMD:C_0603_1608Metric"
 			(at 57.4548 33.02 0)
 			(effects
@@
 			)
 		)
-		(property "Footprint" ""
+		(property "Footprint" "Resistor_SMD:R_0201_0603Metric"
 			(at 177.292 105.41 90)
 			(effects
@@
 			)
 		)
-		(property "Footprint" ""
+		(property "Footprint" "Capacitor_SMD:C_0603_1608Metric"
 			(at 169.2148 85.09 0)
 			(effects
@@
 			)
 		)
-		(property "Footprint" ""
+		(property "Footprint" "B2B-XH-A:CONN_B2B-XH-ALFSN_JST"
 			(at 186.69 33.02 0)
 			(effects
@@
 		)
 		(instances
-			(project ""
+			(project "hammerhead_sensor_module"
 				(path "/5313a223-fa0e-4103-9806-d293f3d5507a/eee24019-9685-4e58-b29e-98c1c045880e"
 					(reference "J9")
@@
 			)
 		)
-		(property "Footprint" ""
+		(property "Footprint" "Resistor_SMD:R_0201_0603Metric"
 			(at 178.562 54.61 90)
 			(effects
@@
 		)
 		(instances
-			(project ""
+			(project "hammerhead_sensor_module"
 				(path "/5313a223-fa0e-4103-9806-d293f3d5507a/eee24019-9685-4e58-b29e-98c1c045880e"
 					(reference "R16")
@@
 			)
 		)
-		(property "Footprint" ""
+		(property "Footprint" "Capacitor_SMD:C_0201_0603Metric"
 			(at 142.24 82.8548 0)
 			(effects
@@
 			)
 		)
-		(property "Footprint" ""
+		(property "Footprint" "Resistor_SMD:R_0201_0603Metric"
 			(at 98.552 149.86 90)
 			(effects
@@
 			)
 		)
-		(property "Footprint" ""
+		(property "Footprint" "ETQP3M4R7KVN:ETQP3M1R0KVN"
 			(at 165.1 129.21 0)
 			(effects
@@
 			)
 		)
-		(property "Footprint" ""
+		(property "Footprint" "Capacitor_SMD:C_0201_0603Metric"
 			(at 70.1548 83.82 0)
 			(effects
@@
 			)
 		)
-		(property "Footprint" ""
+		(property "Footprint" "B2B-XH-A:CONN_B2B-XH-ALFSN_JST"
 			(at 185.42 83.82 0)
 			(effects
@@
 		)
 		(instances
-			(project ""
+			(project "hammerhead_sensor_module"
 				(path "/5313a223-fa0e-4103-9806-d293f3d5507a/eee24019-9685-4e58-b29e-98c1c045880e"
 					(reference "J12")
@@
 			)
 		)
-		(property "Footprint" ""
+		(property "Footprint" "Capacitor_SMD:C_0201_0603Metric"
 			(at 71.4248 33.02 0)
 			(effects
@@
 			)
 		)
-		(property "Footprint" ""
+		(property "Footprint" "ETQP3M4R7KVN:ETQP3M1R0KVN"
 			(at 163.83 180.01 0)
 			(effects
@@
 			)
 		)
-		(property "Footprint" ""
+		(property "Footprint" "Resistor_SMD:R_0201_0603Metric"
 			(at 111.252 149.86 90)
 			(effects
@@
 			)
 		)
-		(property "Footprint" ""
+		(property "Footprint" "TPS92200D1DDCR:DDC0006A_N"
 			(at 115.57 38.1 0)
 			(effects
@@
 		)
 		(instances
-			(project ""
+			(project "hammerhead_sensor_module"
 				(path "/5313a223-fa0e-4103-9806-d293f3d5507a/eee24019-9685-4e58-b29e-98c1c045880e"
 					(reference "U5")
@@
 			)
 		)
-		(property "Footprint" ""
+		(property "Footprint" "Capacitor_SMD:C_0201_0603Metric"
 			(at 143.51 32.0548 0)
 			(effects
@@
 		)
 		(instances
-			(project ""
+			(project "hammerhead_sensor_module"
 				(path "/5313a223-fa0e-4103-9806-d293f3d5507a/eee24019-9685-4e58-b29e-98c1c045880e"
 					(reference "C37")
@@
 			)
 		)
-		(property "Footprint" ""
+		(property "Footprint" "Capacitor_SMD:C_0603_1608Metric"
 			(at 170.4848 34.29 0)
 			(effects
@@
 			)
 		)
-		(property "Footprint" ""
+		(property "Footprint" "Capacitor_SMD:C_0603_1608Metric"
 			(at 56.1848 83.82 0)
 			(effects
@@
 			)
 		)
-		(property "Footprint" ""
+		(property "Footprint" "TPS92200D1DDCR:DDC0006A_N"
 			(at 114.3 88.9 0)
 			(effects
