File: kicad/hammerhead_sensor_module.kicad_pcb (KiCad board)
At the start: 6 copper layers, 87.5 x 58.8 mm, 158 parts, among them IC1 RT6254BHGJ6F, IC3 RT6254BHGJ6F, IC4 MAX98357AETE+T, IC6 TXB0108RGYR, J1 COMMS CONN, J10 12402012E212A, J2 APCI0105-P001A, J3 SMN-303, J4 Conn_01x22_Female, J5 Conn_01x22_Female, J6 Conn_01x03, J7 SM04B-SRSS-TBLFSN, J8 SM04B-SRSS-TBLFSN, J9 B6B-XH-A, SW1 218-2LPSTRF, U1 TPD4E05U06DQAR, U10 TPD4E05U06DQAR, U11 TPD4E05U06DQAR, U12 467651001, U13 RT9742SNGV, U14 TPD4E05U06DQAR, U15 TPD4E05U06DQAR, U16 TPD4E05U06DQAR, U17 TPD4E05U06DQAR, U18 TPD4E05U06DQAR, U19 TPD4E05U06DQAR, U2 MMBT3904TT1G, U3 TLV75733PDBVR, U4 TPD4E05U06DQAR, U5 TPD4E05U06DQAR, U6 TPD4E05U06DQAR, U7 TPD4E05U06DQAR, U8 TPD4E05U06DQAR, U9 TPD4E05U06DQAR

Commit message: generate manufacturing files, final checks, cleanup
Parts:
- added J11: 10164227-1001A1RLF, 10164227-1001A1RLF:101642271001A1RLF, F.Cu at (120.0, 76.0)
- added J12: 10164227-1001A1RLF, 10164227-1001A1RLF:101642271001A1RLF, F.Cu at (120.0, 42.0)
- C8, C9: value 100n -> 0.1uF
- R10, R5: footprint Resistor_SMD:R_0201_0603Metric -> Resistor_SMD:R_0402_1005Metric
- moved C46 0.97 mm to (124.6, 72.7)
- moved R5 0.30 mm to (103.3, 55.5)
- moved R10 0.26 mm to (123.5, 55.5)
Connections:
- R21 pad 2: Net-(Module1A-LED_nACT) -> Net-(J11-LED_nACT)
Routing:
- net Net-(Module1A-LED_nACT): track 4.77 -> 0.00 mm
- net Net-(J11-LED_nACT): track 0.00 -> 4.77 mm
- net 5V: track 4.64 -> 3.89 mm
- net 3.3V: track 30.9 -> 31.5 mm, vias 28 -> 27
- net GND: track 133.9 -> 133.6 mm, vias 353 -> 354
Other:
- board text added: "${REFERENCE}"
