File: kicad/cm5_highspeed.kicad_sch (KiCad schematic)
At the start: 10 parts, among them J16 Conn_01x22_Female, J5 Conn_01x22_Female, U1 467651001, U4 RT9742SNGV

Commit message: finish first pcb revision
Parts:
- removed C33, C34: 100n, Capacitor_SMD:C_0402_1005Metric, symbol Device:C
- removed J16, J5: Conn_01x22_Female, CM5IO:Hirose_FH12-22S-0.5SH_1x22-1MP_P0.50mm_Horizontal, symbol Connector:Conn_01x22_Socket
- removed R22, R23, R24: 2.2K 1%, Resistor_SMD:R_0402_1005Metric, symbol Device:R
- removed U1: 467651001, symbol 467651001:467651001
- removed U4: RT9742SNGV, Package_TO_SOT_SMD:TSOT-23_HandSoldering, symbol CM5IO:RT9742SNGV
- Module1: footprint CM5IO:Raspberry-Pi-5-Compute-Module -> CM5:Raspberry-Pi-5-Compute-Module
Connections:
- net HDMI1_HOTPLUG: now reaches Module1.143 (HDMI1_HOTPLUG)
- net HDMI1_SDA: now reaches Module1.145 (HDMI1_SDA)
- net HDMI1_D2_P: now reaches Module1.146 (HDMI1_TX2_P)
- net HDMI1_SCL: now reaches Module1.147 (HDMI1_SCL)
- net HDMI1_D2_N: now reaches Module1.148 (HDMI1_TX2_N)
- net HDMI1_CEC: now reaches Module1.149 (HDMI1_CEC)
- net HDMI1_D1_P: now reaches Module1.152 (HDMI1_TX1_P)
- net HDMI1_D1_N: now reaches Module1.154 (HDMI1_TX1_N)
- net HDMI1_D0_P: now reaches Module1.158 (HDMI1_TX0_P)
- net HDMI1_D0_N: now reaches Module1.160 (HDMI1_TX0_N)
- net HDMI1_CK_P: now reaches Module1.164 (HDMI1_CLK_P)
- net HDMI1_CK_N: now reaches Module1.166 (HDMI1_CLK_N)
- net HDMI0_CEC: no longer names the net of Module1.151 (HDMI0_CEC)
- net HDMI0_CK_N: no longer names the net of Module1.190 (HDMI0_CLK_N)
- net HDMI0_CK_P: no longer names the net of Module1.188 (HDMI0_CLK_P)
- net HDMI0_D0_N: no longer names the net of Module1.184 (HDMI0_TX0_N)
- net HDMI0_D0_P: no longer names the net of Module1.182 (HDMI0_TX0_P)
- net HDMI0_D1_N: no longer names the net of Module1.178 (HDMI0_TX1_N)
- net HDMI0_D1_P: no longer names the net of Module1.176 (HDMI0_TX1_P)
- net HDMI0_D2_N: no longer names the net of Module1.172 (HDMI0_TX2_N)
- net HDMI0_D2_P: no longer names the net of Module1.170 (HDMI0_TX2_P)
- net HDMI0_HOTPLUG: no longer names the net of Module1.153 (HDMI0_HOTPLUG)
- net HDMI0_SCL: no longer names the net of Module1.200 (HDMI0_SCL)
- net HDMI0_SDA: no longer names the net of Module1.199 (HDMI0_SDA)
- no-connect marks 36 -> 34
Other:
- added sheet hdmi (hdmi.kicad_sch)
- added sheet mipi_csi2_camera_port1 (mipi_csi2_camera_port.kicad_sch)
- added sheet mipi_csi2_camera_port2 (mipi_csi2_camera_port.kicad_sch)
- moved on the sheet: Module1B

Commit message: add docs and cleanup
Changed lines of the file:
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@@
+	(wire
+		(pts
+			(xy 133.35 107.95) (xy 138.43 107.95)
+		)
+		(stroke
+			(width 0)
+			(type default)
+		)
+	)
 	(wire
 		(pts
@@
 	(wire
 		(pts
+			(xy 133.35 184.15) (xy 138.43 184.15)
+		)
+		(stroke
+			(width 0)
+			(type default)
+		)
+	)
+	(wire
+		(pts
 			(xy 30.48 132.08) (xy 33.02 132.08)
 		)
@@
 	(wire
 		(pts
+			(xy 133.35 185.42) (xy 133.35 184.15)
+		)
+		(stroke
+			(width 0)
+			(type default)
+		)
+	)
+	(wire
+		(pts
 			(xy 93.98 109.22) (xy 96.52 109.22)
 		)
@@
 	(wire
 		(pts
-			(xy 133.35 107.95) (xy 138.43 107.95)
-		)
-		(stroke
-			(width 0)
-			(type default)
-		)
-	)
-	(wire
-		(pts
 			(xy 16.51 111.76) (xy 33.02 111.76)
 		)
@@
 	(wire
 		(pts
-			(xy 133.35 184.15) (xy 138.43 184.15)
-		)
-		(stroke
-			(width 0)
-			(type default)
-		)
-	)
-	(wire
-		(pts
 			(xy 93.98 50.8) (xy 138.43 50.8)
 		)
@@
 			(width 0)
 			(type solid)
+		)
+	)
+	(wire
+		(pts
+			(xy 133.35 109.22) (xy 133.35 107.95)
+		)
+		(stroke
+			(width 0)
+			(type default)
 		)
 	)
@@
 	(hierarchical_label "GND"
 		(shape passive)
-		(at 133.35 107.95 180)
+		(at 133.35 109.22 270)
 		(effects
 			(font
@@
 	(hierarchical_label "GND"
 		(shape passive)
-		(at 133.35 184.15 180)
-		(effects
-			(font
+		(at 133.35 185.42 270)
+		(effects
+			(font

Commit message: generate manufacturing files, final checks, cleanup
Parts:
- removed Module1: ComputeModule5-CM5, CM5:Raspberry-Pi-5-Compute-Module, symbol CM5IO:ComputeModule5-CM5
- added J12: 10164227-1001A1RLF, 10164227-1001A1RLF:101642271001A1RLF, symbol 10164227-1001A1RLF:10164227-1001A1RLF
Connections:
- net DPHY0_C_N: now also J12.27 (MIPI0_C_N)
- net DPHY0_C_P: now also J12.29 (MIPI0_C_P)
- net DPHY0_D0_N: now also J12.15 (MIPI0_D0_N)
- net DPHY0_D0_P: now also J12.17 (MIPI0_D0_P)
- net DPHY0_D1_N: now also J12.21 (MIPI0_D1_N)
- net DPHY0_D1_P: now also J12.23 (MIPI0_D1_P)
- net DPHY0_D2_N: now also J12.33 (MIPI0_D2_N)
- net DPHY0_D2_P: now also J12.35 (MIPI0_D2_P)
- net DPHY0_D3_N: now also J12.39 (MIPI0_D3_N)
- net DPHY0_D3_P: now also J12.41 (MIPI0_D3_P)
- net DPHY1_C_N: now also J12.87 (MIPI1_C_N)
- net DPHY1_C_P: now also J12.89 (MIPI1_C_P)
- net DPHY1_D0_N: now also J12.75 (MIPI1_D0_N)
- net DPHY1_D0_P: now also J12.77 (MIPI1_D0_P)
- net DPHY1_D1_N: now also J12.81 (MIPI1_D1_N)
- net DPHY1_D1_P: now also J12.83 (MIPI1_D1_P)
- net DPHY1_D2_N: now also J12.93 (MIPI1_D2_N)
- net DPHY1_D2_P: now also J12.95 (MIPI1_D2_P)
- net DPHY1_D3_N: now also J12.94 (MIPI1_D3_N)
- net DPHY1_D3_P: now also J12.96 (MIPI1_D3_P)
- net GND: now also J12.13 (GND), J12.14 (GND), J12.19 (GND), J12.20 (GND), J12.25 (GND), J12.26 (GND), J12.31 (GND), J12.32 (GND), J12.37 (GND), J12.38 (GND), J12.44 (GND), J12.50 (GND), J12.55 (GND), J12.56 (GND), J12.61 (GND), J12.62 (GND), J12.67 (GND), J12.68 (GND), J12.7 (GND), J12.73 (GND), J12.74 (GND), J12.79 (GND), J12.8 (GND), J12.80 (GND), J12.85 (GND), J12.86 (GND), J12.91 (GND), J12.92 (GND), J12.97 (GND), J12.98 (GND)
- net HDMI1_CEC: now also J12.49 (HDMI1_CEC)
- net HDMI1_CK_N: now also J12.66 (HDMI1_CLK_N)
- net HDMI1_CK_P: now also J12.64 (HDMI1_CLK_P)
- net HDMI1_D0_N: now also J12.60 (HDMI1_TX0_N)
- net HDMI1_D0_P: now also J12.58 (HDMI1_TX0_P)
- net HDMI1_D1_N: now also J12.54 (HDMI1_TX1_N)
- net HDMI1_D1_P: now also J12.52 (HDMI1_TX1_P)
- net HDMI1_D2_N: now also J12.48 (HDMI1_TX2_N)
- net HDMI1_D2_P: now also J12.46 (HDMI1_TX2_P)
- net HDMI1_HOTPLUG: now also J12.43 (HDMI1_HOTPLUG)
- net HDMI1_SCL: now also J12.47 (HDMI1_SCL)
- net HDMI1_SDA: now also J12.45 (HDMI1_SDA)
- net USB2_N: now also J12.3 (USB2_N)
- net USB2_P: now also J12.5 (USB2_P)
- net USB3-0-D_N: now also J12.36 (USB3-0-D_N)
- net USB3-0-D_P: now also J12.34 (USB3-0-D_P)

Commit message: add can controller and transceiver, replace jst connectors with molex micro fit connectors
Changed lines of the file:
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@@
 		)
 	)
-	(hierarchical_label "ID_SD"
+	(hierarchical_label "I2C_SDA_CAM2"
 		(shape input)
 		(at 133.35 175.26 180)
@@
 		)
 	)
-	(hierarchical_label "ID_SC"
+	(hierarchical_label "I2C_SCL_CAM2"
 		(shape input)
 		(at 133.35 172.72 180)
