File: kicad/hdmi.kicad_sch (KiCad schematic)
At the start: 9 parts, among them U1 TPD4E05U06DQAR, U12 467651001, U13 RT9742SNGV, U15 TPD4E05U06DQAR, U5 TPD4E05U06DQAR

Commit message: add docs and cleanup
Other:
- note added: "CM5 has internal pullups"
Changed lines of the file:
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@@
 	(generator_version "9.0")
 	(paper "A4")
+	(text "CM5 has internal pullups"
+		(exclude_from_sim no)
+		(at 193.04 107.696 0)
+		(effects
+			(font
+				(size 1.27 1.27)
+			)
+		)
+	)
 	(text_box "Micro HDMI0"
 		(exclude_from_sim no)
@@
 	)
 	(junction
-		(at 162.56 116.84)
-		(diameter 0)
-		(color 0 0 0 0)
-	)
-	(junction
 		(at 175.26 55.88)
 		(diameter 0)
@@
 	)
 	(junction
+		(at 162.56 111.76)
+		(diameter 0)
+		(color 0 0 0 0)
+	)
+	(junction
 		(at 233.68 31.75)
 		(diameter 0)
@@
 	(wire
 		(pts
-			(xy 162.56 116.84) (xy 204.47 116.84)
+			(xy 162.56 111.76) (xy 204.47 111.76)
 		)
 		(stroke
@@
 	(wire
 		(pts
-			(xy 162.56 66.04) (xy 162.56 116.84)
+			(xy 162.56 66.04) (xy 162.56 111.76)
 		)
 		(stroke
@@
 	(wire
 		(pts
-			(xy 41.91 116.84) (xy 162.56 116.84)
+			(xy 41.91 111.76) (xy 162.56 111.76)
 		)
 		(stroke
@@
 	(hierarchical_label "HDMI_SCL"
 		(shape input)
-		(at 41.91 116.84 180)
-		(effects
-			(font
+		(at 41.91 111.76 180)
+		(effects
+			(font

Commit message: generate manufacturing files, final checks, cleanup
Parts:
- C8, C9: value 100n -> 0.1uF
Changed lines of the file:
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@@
 			)
 		)
-		(property "Value" "100n"
+		(property "Value" "0.1uF"
 			(at 225.171 36.703 0)
 			(effects
@@
 			)
 		)
-		(property "Value" "100n"
+		(property "Value" "0.1uF"
 			(at 192.151 36.703 0)
 			(effects

Commit message: add can controller and transceiver, replace jst connectors with molex micro fit connectors
Connections:
- net TMDS_DATA0+ is gone; now on net HDMI_D0_P: U12.9 (TMDS_DATA0+), U15.2 (D1-)
- net TMDS_DATA0- is gone; now on net HDMI_D0_N: U12.11 (TMDS_DATA0-), U15.1 (D1+)
- net TMDS_DATA2+ is gone; now on net HDMI_D2_P: U12.3 (TMDS_DATA2+), U15.5 (D2-)
- net TMDS_DATA2- is gone; now on net HDMI_D2_N: U12.5 (TMDS_DATA2-), U15.4 (D2+)
