File: kicad/mipi_csi2_camera_port.kicad_sch (KiCad schematic)
At the start: 9 parts, among them J4 Conn_01x22_Female, U11 TPD4E05U06DQAR, U8 TPD4E05U06DQAR, U9 TPD4E05U06DQAR

Commit message: add can controller and transceiver, replace jst connectors with molex micro fit connectors
Connections:
- net C_C_N is gone; now on net C_N: J4.8 (Pin_8), U9.5 (D2-)
- net C_C_P is gone; now on net C_P: J4.9 (Pin_9), U9.4 (D2+)
- net C_D0_N is gone; now on net D0_N: J4.2 (Pin_2), U8.5 (D2-)
- net C_D0_P is gone; now on net D0_P: J4.3 (Pin_3), U8.4 (D2+)
- net C_D1_N is gone; now on net D1_N: J4.5 (Pin_5), U8.2 (D1-)
- net C_D1_P is gone; now on net D1_P: J4.6 (Pin_6), U8.1 (D1+)
- net C_D2_N is gone; now on net D2_N: J4.11 (Pin_11), U9.2 (D1-)
- net C_D2_P is gone; now on net D2_P: J4.12 (Pin_12), U9.1 (D1+)
- net C_D3_N is gone; now on net D3_N: J4.14 (Pin_14), U11.5 (D2-)
- net C_D3_P is gone; now on net D3_P: J4.15 (Pin_15), U11.4 (D2+)
- net CAM_GPIO0: now also J4.17 (Pin_17), U11.2 (D1-)
- net CAM_GPIO1: now also J4.18 (Pin_18), U11.1 (D1+)
