File: kicad/cm5_gpio.kicad_sch (KiCad schematic)
At the start: 24 parts, among them IC4 MAX98357AETE+T, J11 10164227-1001A1RLF, J6 Conn_01x03, J8 BM04B-SRSS-TB_LF__SN_, J9 BM04B-SRSS-TB_LF__SN_, SW1 218-2LPSTRF

Commit message: add board bringup redlines
Connections:
- net 3.3V: no longer C46.1, J11.78 (GPIO_VREF(1.8v/3.3v_Input))
- net 5V: now also J8.1; no longer J8.4
- net GND: now also J8.3; no longer J11.92 (PWR_BUT), J8.2
- net PWM: now also J8.2; no longer J8.3
- net TACHO: now also J8.4; no longer J8.1
- net GPIO_VREF: now reaches J11.84 (+3.3v_(Output)_600mA_Max)
- net GPIO_VREF: now also C46.1, J11.78 (GPIO_VREF(1.8v/3.3v_Input)), J11.86 (+3.3v_(Output)_600mA_Max)
- no-connect marks 34 -> 33
Other:
- note added: "External 3.3V regulator enable signal"
- moved on the sheet: C46
Changed lines of the file:
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@@
 	(generator_version "9.0")
 	(paper "A4")
+	(text "External 3.3V\nregulator enable signal"
+		(exclude_from_sim no)
+		(at 24.638 121.92 0)
+		(effects
+			(font
+				(size 1.27 1.27)
+			)
+		)
+	)
 	(text "TODO: Consider adding\nrtc battery"
 		(exclude_from_sim no)
-		(at 41.402 118.364 0)
+		(at 44.196 118.872 0)
 		(effects
 			(font
@@
 	)
 	(junction
-		(at 118.11 133.35)
+		(at 57.15 133.35)
 		(diameter 0)
 		(color 0 0 0 0)
 	)
 	(junction
-		(at 55.88 143.51)
+		(at 118.11 133.35)
 		(diameter 0)
 		(color 0 0 0 0)
@@
 	)
 	(junction
-		(at 24.13 125.73)
+		(at 26.67 125.73)
 		(diameter 0)
 		(color 0 0 0 0)
@@
 	)
 	(junction
+		(at 54.61 125.73)
+		(diameter 0)
+		(color 0 0 0 0)
+	)
+	(junction
 		(at 55.88 80.01)
 		(diameter 1.016)
@@
 	)
 	(no_connect
-		(at 57.15 135.89)
-	)
-	(no_connect
 		(at 118.11 41.91)
 	)
@@
 	)
 	(no_connect
-		(at 57.15 133.35)
+		(at 118.11 120.65)
 	)
 	(no_connect
-		(at 118.11 120.65)
+		(at 57.15 143.51)
 	)
 	(no_connect
@@
 	(wire
 		(pts
-			(xy 55.88 120.65) (xy 55.88 143.51)
+			(xy 55.88 120.65) (xy 55.88 151.13)
 		)
 		(stroke
@@
 	(wire
 		(pts
-			(xy 55.88 143.51) (xy 55.88 151.13)
-		)
-		(stroke
-			(width 0)
-			(type solid)
-		)
-	)
-	(wire
-		(pts
 			(xy 189.23 62.23) (xy 190.5 62.23)
 		)
@@
 	(wire
 		(pts
+			(xy 54.61 125.73) (xy 54.61 133.35)
+		)
+		(stroke
+			(width 0)
+			(type default)
+		)
+	)
+	(wire
+		(pts
 			(xy 119.38 69.85) (xy 119.38 82.55)
 		)
@@
 	(wire
 		(pts
+			(xy 57.15 133.35) (xy 57.15 135.89)
+		)
+		(stroke
+			(width 0)
+			(type default)
+		)
+	)
+	(wire
+		(pts
 			(xy 55.88 67.31) (xy 55.88 80.01)
 		)
@@
 	(wire
 		(pts
-			(xy 24.13 133.35) (xy 24.13 135.89)
+			(xy 26.67 133.35) (xy 26.67 135.89)
 		)
 		(stroke
@@
 	(wire
 		(pts
-			(xy 24.13 121.92) (xy 24.13 125.73)
-		)
-		(stroke
-			(width 0)
-			(type solid)
-		)
-	)
-	(wire
-		(pts
 			(xy 194.31 124.46) (xy 194.31 128.27)
 		)
@@
 	(wire
 		(pts
-			(xy 229.87 97.79) (xy 236.22 97.79)
+			(xy 57.15 125.73) (xy 54.61 125.73)
 		)
 		(stroke
@@
 	(wire
 		(pts
-			(xy 43.18 128.27) (xy 57.15 128.27)
+			(xy 229.87 97.79) (xy 236.22 97.79)
 		)
 		(stroke
 			(width 0)
-			(type solid)
+			(type default)
 		)
 	)
@@
 	(wire
 		(pts
-			(xy 43.18 130.81) (xy 57.15 130.81)
-		)
-		(stroke
-			(width 0)
-			(type solid)
-		)
-	)
-	(wire
-		(pts
 			(xy 189.23 54.61) (xy 189.23 59.69)
 		)
@@
 	(wire
 		(pts
+			(xy 43.18 130.81) (xy 57.15 130.81)
+		)
+		(stroke
+			(width 0)
+			(type default)
+		)
+	)
+	(wire
+		(pts
 			(xy 261.62 53.34) (xy 264.16 53.34)
 		)
@@
 	(wire
 		(pts
+			(xy 43.18 128.27) (xy 57.15 128.27)
+		)
+		(stroke
+			(width 0)
+			(type default)
+		)
+	)
+	(wire
+		(pts
 			(xy 236.22 97.79) (xy 236.22 99.06)
 		)
@@
 	(wire
 		(pts
-			(xy 130.81 97.79) (xy 118.11 97.79)
+			(xy 54.61 133.35) (xy 57.15 133.35)
 		)
 		(stroke
@@
 	(wire
 		(pts
-			(xy 55.88 143.51) (xy 57.15 143.51)
+			(xy 130.81 97.79) (xy 118.11 97.79)
 		)
 		(stroke
@@
 	(wire
 		(pts
-			(xy 24.13 125.73) (xy 57.15 125.73)
-		)
-		(stroke
-			(width 0)
-			(type solid)
-		)
-	)
-	(wire
-		(pts
 			(xy 66.04 179.07) (xy 71.12 179.07)
 		)
@@
 	(wire
 		(pts
+			(xy 24.13 125.73) (xy 26.67 125.73)
+		)
+		(stroke
+			(width 0)
+			(type default)
+		)
+	)
+	(wire
+		(pts
 			(xy 118.11 148.59) (xy 146.05 148.59)
 		)
@@
 		)
 	)
+	(wire
+		(pts
+			(xy 26.67 125.73) (xy 54.61 125.73)
+		)
+		(stroke
+			(width 0)
+			(type default)
+		)
+	)
 	(label "PCM_DOUT"
 		(at 208.28 163.83 180)
@@
 	)
 	(label "SCL0"
-		(at 54.61 128.27 180)
+		(at 52.07 128.27 180)
 		(effects
 			(font
@@
 	)
 	(label "SDA0"
-		(at 54.61 130.81 180)
+		(at 52.07 130.81 180)
 		(effects
 			(font
@@
 	(hierarchical_label "GND"
 		(shape passive)
-		(at 24.13 135.89 270)
+		(at 26.67 135.89 270)
 		(effects
 			(font
@@
 		)
 	)
-	(hierarchical_label "3.3V"
+	(hierarchical_label "5V"
 		(shape input)
-		(at 24.13 121.92 90)
+		(at 184.15 25.4 90)
 		(effects
 			(font
@@
 		)
 	)
-	(hierarchical_label "5V"
-		(shape input)
-		(at 184.15 25.4 90)
+	(hierarchical_label "GPIO_VREF"
+		(shape output)
+		(at 24.13 125.73 180)
 		(effects
 			(font
 				(size 1.27 1.27)
 			)
-			(justify left)
+			(justify right)
 		)
 	)
@@
 	(symbol
 		(lib_id "Device:C")
-		(at 24.13 129.54 0)
+		(at 26.67 129.54 0)
 		(unit 1)
 		(exclude_from_sim no)
@@
 		(fields_autoplaced yes)
 		(property "Reference" "C46"
-			(at 27.94 128.2699 0)
+			(at 30.48 128.2699 0)
 			(effects
 				(font
@@
 		)
 		(property "Value" "0.1uF"
-			(at 27.94 130.8099 0)
+			(at 30.48 130.8099 0)
 			(effects
 				(font
@@
 		)
 		(property "Footprint" "Capacitor_SMD:C_0201_0603Metric"
-			(at 25.0952 133.35 0)
+			(at 27.6352 133.35 0)
 			(effects
 				(font
@@
 		)
 		(property "Datasheet" "~"
-			(at 24.13 129.54 0)
+			(at 26.67 129.54 0)
 			(effects
 				(font
@@
 		)
 		(property "Description" "Unpolarized capacitor"
-			(at 24.13 129.54 0)
+			(at 26.67 129.54 0)
 			(effects
 				(font
@@
 		)
 		(property "DigiKey_Part_Number" ""
-			(at 24.13 129.54 0)
+			(at 26.67 129.54 0)
 			(effects
 				(font
@@
 		)
 		(property "Purchase-URL" ""
-			(at 24.13 129.54 0)
+			(at 26.67 129.54 0)
 			(effects
 				(font
