File: kicad/power.kicad_sch (KiCad schematic)
At the start: 32 parts, among them IC1 RT6254BHGJ6F, IC3 RT6254BHGJ6F, U3 TLV75733PDBVR

Commit message: finish first pcb revision
Parts:
- C1, C4: footprint (none) -> 25TQC100MD3:16TDC150MYF
- C26, C3: footprint (none) -> 10TPE220ML:16TDC150MYF
- C30, C32: footprint (none) -> Capacitor_SMD:C_0201_0603Metric
- FB1: footprint (none) -> BLM21PG300SN1D:BEADC2012X105N
- IC1, IC3: footprint (none) -> RT6254BHGJ6F:SOT95P280X100-6N
- L1, L3: footprint (none) -> ETQP3M4R7KVN:ETQP3M1R0KVN
- U3: footprint (none) -> TLV75733PDBVR:DBV0005A_N
Changed lines of the file:
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@@
 			)
 		)
-		(property "Footprint" ""
+		(property "Footprint" "RT6254BHGJ6F:SOT95P280X100-6N"
 			(at 120.65 205.41 0)
 			(effects
@@
 			)
 		)
-		(property "Footprint" ""
+		(property "Footprint" "RT6254BHGJ6F:SOT95P280X100-6N"
 			(at 120.65 144.45 0)
 			(effects
@@
 		)
 		(instances
-			(project ""
+			(project "hammerhead_sensor_module"
 				(path "/5313a223-fa0e-4103-9806-d293f3d5507a/8293f066-7499-4d50-94d4-999fc085e2c1"
 					(reference "IC1")
@@
 			)
 		)
-		(property "Footprint" ""
+		(property "Footprint" "25TQC100MD3:16TDC150MYF"
 			(at -46.66 58.42 0)
 			(effects
@@
 		)
 		(instances
-			(project ""
+			(project "hammerhead_sensor_module"
 				(path "/5313a223-fa0e-4103-9806-d293f3d5507a/8293f066-7499-4d50-94d4-999fc085e2c1"
 					(reference "C1")
@@
 			)
 		)
-		(property "Footprint" ""
+		(property "Footprint" "BLM21PG300SN1D:BEADC2012X105N"
 			(at 318.44 93.98 0)
 			(effects
@@
 		)
 		(instances
-			(project ""
+			(project "hammerhead_sensor_module"
 				(path "/5313a223-fa0e-4103-9806-d293f3d5507a/8293f066-7499-4d50-94d4-999fc085e2c1"
 					(reference "FB1")
@@
 			)
 		)
-		(property "Footprint" ""
+		(property "Footprint" "ETQP3M4R7KVN:ETQP3M1R0KVN"
 			(at 160.02 206.68 0)
 			(effects
@@
 			)
 		)
-		(property "Footprint" ""
+		(property "Footprint" "ETQP3M4R7KVN:ETQP3M1R0KVN"
 			(at 160.02 145.72 0)
 			(effects
@@
 		)
 		(instances
-			(project ""
+			(project "hammerhead_sensor_module"
 				(path "/5313a223-fa0e-4103-9806-d293f3d5507a/8293f066-7499-4d50-94d4-999fc085e2c1"
 					(reference "L1")
@@
 			)
 		)
-		(property "Footprint" ""
+		(property "Footprint" "TLV75733PDBVR:DBV0005A_N"
 			(at 111.76 170.18 0)
 			(effects
@@
 		)
 		(instances
-			(project ""
+			(project "hammerhead_sensor_module"
 				(path "/5313a223-fa0e-4103-9806-d293f3d5507a/8293f066-7499-4d50-94d4-999fc085e2c1"
 					(reference "U3")
@@
 			)
 		)
-		(property "Footprint" ""
+		(property "Footprint" "Capacitor_SMD:C_0201_0603Metric"
 			(at 88.5952 170.18 0)
 			(effects
@@
 		)
 		(instances
-			(project ""
+			(project "hammerhead_sensor_module"
 				(path "/5313a223-fa0e-4103-9806-d293f3d5507a/8293f066-7499-4d50-94d4-999fc085e2c1"
 					(reference "C30")
@@
 			)
 		)
-		(property "Footprint" ""
+		(property "Footprint" "25TQC100MD3:16TDC150MYF"
 			(at -46.66 119.38 0)
 			(effects
@@
 			)
 		)
-		(property "Footprint" ""
+		(property "Footprint" "Capacitor_SMD:C_0201_0603Metric"
 			(at 129.2352 170.18 0)
 			(effects
@@
 			)
 		)
-		(property "Footprint" ""
+		(property "Footprint" "10TPE220ML:16TDC150MYF"
 			(at 127.33 58.42 0)
 			(effects
@@
 		)
 		(instances
-			(project ""
+			(project "hammerhead_sensor_module"
 				(path "/5313a223-fa0e-4103-9806-d293f3d5507a/8293f066-7499-4d50-94d4-999fc085e2c1"
 					(reference "C3")
@@
 			)
 		)
-		(property "Footprint" ""
+		(property "Footprint" "10TPE220ML:16TDC150MYF"
 			(at 142.57 119.38 0)
 			(effects

Commit message: add docs and cleanup
Other:
- moved on the sheet: C1, C10, C12, C14, C16, C17, C18, C21, C22, C23, C24, C25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

Commit message: generate manufacturing files, final checks, cleanup
Parts:
- R10, R5: footprint Resistor_SMD:R_0201_0603Metric -> Resistor_SMD:R_0402_1005Metric
Changed lines of the file:
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@@
 			)
 		)
-		(property "Footprint" "Resistor_SMD:R_0201_0603Metric"
+		(property "Footprint" "Resistor_SMD:R_0402_1005Metric"
 			(at 153.162 102.87 90)
 			(effects
@@
 			)
 		)
-		(property "Footprint" "Resistor_SMD:R_0201_0603Metric"
+		(property "Footprint" "Resistor_SMD:R_0402_1005Metric"
 			(at 155.702 45.72 90)
 			(effects

Commit message: add board bringup redlines
Parts:
- added R1: 10k, Resistor_SMD:R_0201_0603Metric, symbol Device:R
Connections:
- net 5V: no longer U3.3 (EN)
- net GND: now also R1.1
- new net 3.3V_EN: R1.2, U3.3 (EN)
Other:
- moved on the sheet: C30
Changed lines of the file:
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@@
 	)
 	(junction
-		(at 72.39 151.13)
+		(at 59.69 151.13)
 		(diameter 0)
 		(color 0 0 0 0)
@@
 	)
 	(junction
-		(at 58.42 106.68)
+		(at 81.28 158.75)
 		(diameter 0)
 		(color 0 0 0 0)
 	)
 	(junction
-		(at 195.58 39.37)
+		(at 58.42 106.68)
 		(diameter 0)
 		(color 0 0 0 0)
 	)
 	(junction
-		(at 166.37 96.52)
+		(at 195.58 39.37)
 		(diameter 0)
 		(color 0 0 0 0)
 	)
 	(junction
-		(at 83.82 151.13)
+		(at 166.37 96.52)
 		(diameter 0)
 		(color 0 0 0 0)
@@
 	(wire
 		(pts
-			(xy 64.77 151.13) (xy 72.39 151.13)
+			(xy 52.07 151.13) (xy 59.69 151.13)
 		)
 		(stroke
@@
 	(wire
 		(pts
-			(xy 72.39 151.13) (xy 83.82 151.13)
+			(xy 59.69 151.13) (xy 83.82 151.13)
 		)
 		(stroke
@@
 	(wire
 		(pts
+			(xy 81.28 158.75) (xy 83.82 158.75)
+		)
+		(stroke
+			(width 0)
+			(type default)
+		)
+	)
+	(wire
+		(pts
 			(xy 157.48 54.61) (xy 157.48 58.42)
 		)
@@
 	(wire
 		(pts
-			(xy 81.28 96.52) (xy 73.66 96.52)
+			(xy 76.2 158.75) (xy 81.28 158.75)
 		)
 		(stroke
@@
 	(wire
 		(pts
-			(xy 166.37 96.52) (xy 179.07 96.52)
+			(xy 81.28 96.52) (xy 73.66 96.52)
 		)
 		(stroke
@@
 	(wire
 		(pts
-			(xy 83.82 151.13) (xy 83.82 158.75)
+			(xy 166.37 96.52) (xy 179.07 96.52)
 		)
 		(stroke
@@
 	(wire
 		(pts
+			(xy 81.28 158.75) (xy 81.28 160.02)
+		)
+		(stroke
+			(width 0)
+			(type default)
+		)
+	)
+	(wire
+		(pts
 			(xy 124.46 39.37) (xy 128.27 39.37)
 		)
@@
 	(wire
 		(pts
+			(xy 81.28 167.64) (xy 81.28 168.91)
+		)
+		(stroke
+			(width 0)
+			(type default)
+		)
+	)
+	(wire
+		(pts
 			(xy 58.42 99.06) (xy 58.42 96.52)
 		)
@@
 	(wire
 		(pts
-			(xy 72.39 158.75) (xy 72.39 161.29)
+			(xy 59.69 158.75) (xy 59.69 161.29)
 		)
 		(stroke
@@
 		)
 	)
+	(hierarchical_label "3.3V_EN"
+		(shape input)
+		(at 76.2 158.75 180)
+		(effects
+			(font
+				(size 1.27 1.27)
+			)
+			(justify right)
+		)
+	)
+	(hierarchical_label "GND"
+		(shape passive)
+		(at 81.28 168.91 270)
+		(effects
+			(font
+				(size 1.27 1.27)
+			)
+			(justify right)
+		)
+	)
 	(hierarchical_label "14.8V"
 		(shape input)
@@
 	(hierarchical_label "5V"
 		(shape output)
-		(at 64.77 151.13 180)
+		(at 52.07 151.13 180)
 		(effects
 			(font
@@
 	(hierarchical_label "GND"
 		(shape passive)
-		(at 72.39 161.29 270)
+		(at 59.69 161.29 270)
 		(effects
 			(font
@@
 	(symbol
 		(lib_id "Device:C")
-		(at 72.39 154.94 0)
+		(at 59.69 154.94 0)
 		(unit 1)
 		(exclude_from_sim no)
@@
 		(fields_autoplaced yes)
 		(property "Reference" "C30"
-			(at 76.2 153.6699 0)
+			(at 63.5 153.6699 0)
 			(effects
 				(font
@@
 		)
 		(property "Value" "1uF"
-			(at 76.2 156.2099 0)
+			(at 63.5 156.2099 0)
 			(effects
 				(font
@@
 		)
 		(property "Footprint" "Capacitor_SMD:C_0201_0603Metric"
-			(at 73.3552 158.75 0)
+			(at 60.6552 158.75 0)
 			(effects
 				(font
@@
 		)
 		(property "Datasheet" "~"
-			(at 72.39 154.94 0)
+			(at 59.69 154.94 0)
 			(effects
 				(font
@@
 		)
 		(property "Description" "Unpolarized capacitor"
-			(at 72.39 154.94 0)
+			(at 59.69 154.94 0)
 			(effects
 				(font
@@
 		)
 		(property "DigiKey_Part_Number" ""
-			(at 72.39 154.94 0)
+			(at 59.69 154.94 0)
 			(effects
 				(font
@@
 		)
 		(property "Purchase-URL" ""
-			(at 72.39 154.94 0)
+			(at 59.69 154.94 0)
 			(effects
 				(font
@@
 					(unit 1)
 				)
+			)
+		)
+	)
+	(symbol
+		(lib_id "Device:R")
+		(at 81.28 163.83 180)
+		(unit 1)
+		(exclude_from_sim no)
+		(in_bom yes)
+		(on_board yes)
+		(dnp no)
+		(fields_autoplaced yes)
+		(property "Reference" "R1"
+			(at 83.82 162.5599 0)
+			(effects
+				(font
+					(size 1.27 1.27)
+				)
+				(justify right)
+			)
+		)
+		(property "Value" "10k"
+			(at 83.82 165.0999 0)
+			(effects
+				(font
+					(size 1.27 1.27)
+				)
+				(justify right)
+			)
+		)
+		(property "Footprint" "Resistor_SMD:R_0201_0603Metric"
+			(at 83.058 163.83 90)
+			(effects
+				(font
+					(size 1.27 1.27)
+				)
+				(hide yes)
+			)
+		)
+		(property "Datasheet" "~"
+			(at 81.28 163.83 0)
+			(effects
+				(font
+					(size 1.27 1.27)
+				)
+				(hide yes)
+			)
+		)
+		(property "Description" "Resistor"
+			(at 81.28 163.83 0)
+			(effects
+				(font
+					(size 1.27 1.27)
+				)
+				(hide yes)
+			)
+		)
+		(property "DigiKey_Part_Number" ""
+			(at 81.28 163.83 0)
+			(effects
+				(font
+					(size 1.27 1.27)
+				)
+				(hide yes)
+			)
+		)
+		(property "Purchase-URL" ""
+			(at 81.28 163.83 0)
+			(effects
+				(font
+					(size 1.27 1.27)
+				)
+				(hide yes)
+			)
+		)
+		(pin "2"
+		)
+		(pin "1"
+		)
+		(instances
+			(project "hammerhead_sensor_module"
+				(path "/5313a223-fa0e-4103-9806-d293f3d5507a/8293f066-7499-4d50-94d4-999fc085e2c1"
+					(reference "R1")
+					(unit 1)
+				)
